Commit message: mycobot_1

File: mycobot_description/urdf/mech/adaptive_gripper.urdf.xacro (robot description, xacro)
@@ -47,4 +47,20 @@
       <xacro:insert_block name="origin"/>
     </joint>
+    <!-- EE_link: End Effector frame at the gripper tip (for closed gripper). Adjust origin as needed in RViz. -->
+    <link name="${prefix}EE_link">
+      <!-- Minimal inertial values to keep simulators happy if needed; can be removed if only kinematic. -->
+      <inertial>
+        <origin xyz="0 0 0" rpy="0 0 0"/>
+        <mass value="0.001"/>
+        <inertia ixx="1e-7" ixy="0" ixz="0" iyy="1e-7" iyz="0" izz="1e-7"/>
+      </inertial>
+      <!-- No visual/collision by default to avoid affecting collisions. -->
+    </link>
+    <joint name="${prefix}gripper_base_to_${prefix}EE_link" type="fixed">
+      <parent link="${prefix}gripper_base"/>
+      <child link="${prefix}EE_link"/>
+      <!-- Initial guess: along +Y from gripper_base; refine xyz/rpy after viewing in RViz. -->
+      <origin xyz="0.0 0.085 0.0" rpy="0 0 0"/>
+    </joint>
     <link name="${prefix}gripper_left1">
       <xacro:gripper_link_inertial/>

File: mycobot_description/urdf/robots/mycobot_280.urdf.xacro (robot description, xacro)
@@ -54,3 +54,6 @@
       use_gazebo="$(arg use_gazebo)"/>
     <xacro:include filename="$(find mycobot_description)/urdf/sensors/intel_rgbd_cam_d435.urdf.xacro"/>
+    <!-- Note: Contact sensors removed - use simple_collision_detector.py instead -->
+    <!-- The Gazebo contact sensors don't work properly with ROS2 Jazzy + Gazebo Harmony -->
+    <!-- Use: ros2 run mycobot_description simple_collision_detector.py -->
 </robot>
